File: hardware/PID.kicad_sch (KiCad schematic)
At the start: 20 parts, among them J1 USB_C_Receptacle_USB2.0_16P, SW1 SW_MMI_Q5-100, SW2 SW_MMI_Q5-100, SW3 SW_MMI_Q5-100, SW4 SW_MMI_Q5-100, SW5 SW_MMI_Q5-100, SW6 SW_MMI_Q5-100, U1 TCA9548APWR, U2 LT1962-3.3, U3 RP2040

Commit message: Sche
Other:
- note added: "diy_stream_deck"
Changed lines of the file:
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@@
 	(generator_version "10.0")
 	(paper "A4")
+	(text "diy_stream_deck\n"
+		(exclude_from_sim no)
+		(at 193.04 175.26 0)
+		(effects
+			(font
+				(size 2.54 2.54)
+			)
+		)
+	)
 	(junction
 		(at 60.96 49.53)
